File: avrboard.kicad_pcb (KiCad board)
At the start: 2 copper layers, 45.1 x 62.9 mm, 21 parts, among them IC1 ATMEGA328P-P, P1 FTDI, P2 ICSP, SW1 RESET, X1 16MHz

Commit message: Include a caption on the back silkscreen.
OSH Park refuses to accept an empty back silkscreen layer, for some
reason.
Other:
- board text added: "AVR PROGRAMMING AND DEVELOPMENT BOARD"
Changed lines of the file:
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@@
     (area 121.806305 33.604999 167.904886 96.5835)
     (thickness 1.6)
-    (drawings 62)
+    (drawings 63)
     (tracks 200)
     (zones 0)
@@
     )
   )
+  (gr_text "AVR PROGRAMMING\nAND DEVELOPMENT\nBOARD" (at 151.765 81.915) (layer B.SilkS)
+    (effects (font (size 1.016 1.016) (thickness 0.254)) (justify mirror))
+  )
   (gr_line (start 122.555 36.83) (end 122.555 34.925) (angle 90) (layer Edge.Cuts) (width 0.1))
